Commit message: add walls detect

File: velodyne_simulator/velodyne_description/urdf/example.urdf.xacro (robot description, xacro)
@@ -26,5 +26,5 @@
     <inertial>
       <origin xyz="0 0 0"/>
-      <mass value="10"/>
+      <mass value="100"/>
       <inertia ixx="3.0" ixy="0.0" ixz="0.0"
                iyy="3.0" iyz="0.0"

Commit message: add factory gzWorld

File: velodyne_simulator/velodyne_description/urdf/example.urdf.xacro (robot description, xacro)
@@ -13,4 +13,8 @@
     <origin xyz="0 0 0.05" rpy="0 0 0" />
   </joint>
+  <gazebo reference="base_link">
+    <material>Gazebo/Red</material>
+    <turnGravityOff>false</turnGravityOff>
+  </gazebo>
   <link name="base_link" >
     <visual>
@@ -26,5 +30,5 @@
     <inertial>
       <origin xyz="0 0 0"/>
-      <mass value="100"/>
+      <mass value="10"/>
       <inertia ixx="3.0" ixy="0.0" ixz="0.0"
                iyy="3.0" iyz="0.0"
